Commit message: modified window size and location

File: mtconnect_example/mtconnect_cnc_robot_example/urdf/mtconnect_irb2400_cnc_environment.xacro (robot description, xacro)
@@ -10,8 +10,8 @@
 	<!-- parameters -->
 	<xacro:property name="platform_thickness" value="0.1"/>
-	<xacro:property name="window_width" value="0.32"/>
-	<xacro:property name="window_length" value="0.32"/>
-	<xacro:property name="window_frame_thickness" value="0.4"/>
-	<xacro:property name="window_frame_depth" value="0.2"/>
+	<xacro:property name="window_width" value="0.40"/>
+	<xacro:property name="window_length" value="0.40"/>
+	<xacro:property name="window_frame_thickness" value="0.32"/>
+	<xacro:property name="window_frame_depth" value="1.0"/>
 	<!-- color definitions -->
         <material name="blue">
@@ -105,5 +105,5 @@
 	</joint>
 	<joint name="world_to_window" type="fixed">
-		<origin xyz="1.6 0.40 0.8" rpy="0 1.5708 0"/>
+		<origin xyz="2.0 0.40 0.8" rpy="0 1.5708 0"/>
 		<parent link="world_frame"/>
 		<child link="window_frame"/>

Commit message: Changed filters in order to reduce wrist motion.  Created special environment server launch with gdb call in order to track down an issue.

File: mtconnect_example/mtconnect_cnc_robot_example/urdf/mtconnect_irb2400_cnc_environment.xacro (robot description, xacro)
@@ -73,4 +73,5 @@
 	<!-- link definitions -->
 	<link name="world_frame"/>
+	<link name="palm_intermediate"/>
 	<!--link name="palm"/-->
 	<link name="tcp_frame"/>
@@ -91,4 +92,13 @@
 		</collision>
 	</link>
+	<link name="robot_rear_wall_link">
+		<collision>
+			<origin xyz="0 1 0" rpy="0 0 0"/>
+			<geometry>
+				<box size="0.25 2.0 2.0"/>
+			</geometry>
+			<material name="red"/>
+		</collision>
+	</link>
 	<xacro:window_links w="${window_width}" l="${window_length}"
 		t="${window_frame_thickness}" d="${window_frame_depth}"/>
@@ -98,4 +108,9 @@
 		<parent link="world_frame"/>
 		<child link="robot_platform_link"/>
+	</joint>
+	<joint name="world_to_robot_rear_wall" type ="fixed">
+		<origin xyz="-0.5 -1.0 1.0" rpy="0 0 0"/>
+		<parent link="world_frame"/>
+		<child link="robot_rear_wall_link"/>
 	</joint>
 	<joint name="platform_to_base_joint" type ="fixed">
@@ -109,7 +124,12 @@
 		<child link="window_frame"/>
 	</joint>
-	<joint name="tool_to_palm" type="fixed">
+	<joint name="tool_to_palm_intermediate" type="fixed">
 		<origin xyz="0.08 0 0" rpy="0 1.5708 0"/>
 		<parent link="tool0"/>
+		<child link="palm_intermediate"/>
+	</joint>
+	<joint name="palm_intermediate_to_palm" type="fixed">
+		<origin xyz="0 0 0" rpy="0 0 0.52"/>
+		<parent link="palm_intermediate"/>
 		<child link="${robotiq_prefix}palm"/>
 	</joint>

Commit message: modified the dimensions of the cnc window

File: mtconnect_example/mtconnect_cnc_robot_example/urdf/mtconnect_irb2400_cnc_environment.xacro (robot description, xacro)
@@ -10,7 +10,7 @@
 	<!-- parameters -->
 	<xacro:property name="platform_thickness" value="0.1"/>
-	<xacro:property name="window_width" value="0.40"/>
-	<xacro:property name="window_length" value="0.40"/>
-	<xacro:property name="window_frame_thickness" value="0.32"/>
+	<xacro:property name="window_width" value="0.52"/>
+	<xacro:property name="window_length" value="0.52"/>
+	<xacro:property name="window_frame_thickness" value="0.20"/>
 	<xacro:property name="window_frame_depth" value="1.0"/>
 	<!-- color definitions -->
@@ -125,5 +125,5 @@
 	</joint>
 	<joint name="tool_to_palm_intermediate" type="fixed">
-		<origin xyz="0.08 0 0" rpy="0 1.5708 0"/>
+		<origin xyz="0.165 0 0" rpy="0 1.5708 0"/>
 		<parent link="tool0"/>
 		<child link="palm_intermediate"/>
