Commit message: modified arm_group instances to 'm16i20b' instead of 'manipulator'

File: mtconnect_example/mtconnect_cnc_robot_example/urdf/mtconnect_m16ib20_cnc_environment.xacro (robot description, xacro)
@@ -11,5 +11,5 @@
 	<xacro:property name="window_length" value="0.32"/>
 	<xacro:property name="window_frame_thickness" value="0.4"/>
-	<xacro:property name="window_frame_depth" value="0.2"/>
+	<xacro:property name="window_frame_depth" value="1.0"/>
 	<!-- color definitions -->
         <material name="blue">
@@ -103,5 +103,5 @@
 	</joint>
 	<joint name="world_to_window" type="fixed">
-		<origin xyz="1.6 0.4 0.8" rpy="0 1.5708 0"/>
+		<origin xyz="2.0 0.4 0.8" rpy="0 1.5708 0"/>
 		<parent link="world_frame"/>
 		<child link="window_frame"/>

Commit message: uses prefix for robotiq gripper components

File: mtconnect_example/mtconnect_cnc_robot_example/urdf/mtconnect_m16ib20_cnc_environment.xacro (robot description, xacro)
@@ -3,6 +3,8 @@
 	<include filename="$(find fanuc_config)/urdf/M16iB20_macro.xacro"/>
 	<include filename="$(find robotiq_s_model_visualization)/cfg/s-model_mesh_macro.xacro" />
+	<!-- prefixes -->
+	<xacro:property name="robotiq_prefix" value="robotiq_"/>
 	<!-- instantiating xacros -->
-	<xacro:s-model_mesh prefix=""/>
+	<xacro:s-model_mesh prefix="${robotiq_prefix}"/>
 	<xacro:M16iB20 prefix=""/>
 	<!-- parameters -->
@@ -110,9 +112,9 @@
 		<origin xyz="0.165 0 0" rpy="0 1.5708 0"/>
 		<parent link="tool0"/>
-		<child link="palm"/>
+		<child link="${robotiq_prefix}palm"/>
 	</joint>
 	<joint name="palm_to_tcp" type="fixed">
 		<origin xyz="0 0 0" rpy="0 0 0"/>
-		<parent link="palm"/>
+		<parent link="${robotiq_prefix}palm"/>
 		<child link="tcp_frame"/>
 	</joint>

Commit message: added configuration and launch files for m16ib20

File: mtconnect_example/mtconnect_cnc_robot_example/urdf/mtconnect_m16ib20_cnc_environment.xacro (robot description, xacro)
@@ -10,7 +10,7 @@
 	<!-- parameters -->
 	<xacro:property name="platform_thickness" value="0.1"/>
-	<xacro:property name="window_width" value="0.32"/>
-	<xacro:property name="window_length" value="0.32"/>
-	<xacro:property name="window_frame_thickness" value="0.4"/>
+	<xacro:property name="window_width" value="0.52"/>
+	<xacro:property name="window_length" value="0.52"/>
+	<xacro:property name="window_frame_thickness" value="0.2"/>
 	<xacro:property name="window_frame_depth" value="1.0"/>
 	<!-- color definitions -->

Commit message: Updated m16iB20 with cnc model.  Changed pick/load locations and urdf to accomadate new cnc model

File: mtconnect_example/mtconnect_cnc_robot_example/urdf/mtconnect_m16ib20_cnc_environment.xacro (robot description, xacro)
@@ -91,4 +91,12 @@
 		</collision>
 	</link>
+	<link name="cnc_link">
+		<visual>
+			<geometry>
+        <mesh filename="package://mtconnect_cnc_robot_example/meshes/cnc_lathe.STL"/>
+			</geometry>
+			<material name="red"/>
+		</visual>
+	</link>
 	<xacro:window_links w="${window_width}" l="${window_length}"
 		t="${window_frame_thickness}" d="${window_frame_depth}"/>
@@ -98,4 +106,9 @@
 		<parent link="world_frame"/>
 		<child link="robot_platform_link"/>
+	</joint>
+	<joint name="world_to_cnc_joint" type ="fixed">
+		<origin xyz="2.6 1.325 -0.45" rpy="1.5708 0 -1.5708"/>
+		<parent link="world_frame"/>
+		<child link="cnc_link"/>
 	</joint>
 	<joint name="platform_to_base_joint" type ="fixed">
