Commit message: URDF modifications to show CNC and robot tool in Rviz.  Added associated state publishers to main launch file

File: mtconnect_example/mtconnect_example_launch/urdf/mtconnect_m16ib20_demo_env.urdf (robot description, URDF)
Before this commit: robot NIST_Robot, 7 links, 5 joints
Links:
- removed link end_effector_link
- removed link tcp_frame
- removed link tool0
Joints:
- removed joint tool_to_end_effector
- removed joint tool_to_tcp

File: mtconnect_example/mtconnect_example_launch/urdf/mtconnect_m16ib20_demo_env.xacro (robot description, xacro)
@@ -1,9 +1,6 @@
 <?xml version="1.0" ?>
 <robot name="NIST_Robot" xmlns:xacro="http://ros.org/wiki/xacro">
-	<include filename="$(find fanuc_config)/urdf/M16iB20_macro.xacro"/>
 	<!-- parameters -->
 	<xacro:property name="platform_thickness" value="0.1"/>
-	<xacro:property name="end_effector_length" value="0.35"/>
-	<xacro:property name="end_effector_diameter" value="0.1"/>
 	<!-- color definitions -->
   <material name="blue">
@@ -24,9 +21,6 @@
   <!-- robot definitions, also defined in robot urdf -->
 	<link name="base_link"/>
-	<link name="tool0"/>
 	<!-- link definitions -->
 	<link name="world_frame"/>
-	<!--link name="palm"/-->
-	<link name="tcp_frame"/>
 	<link name="robot_platform_link">
 		<visual>
@@ -36,13 +30,4 @@
 			</geometry>
 			<material name="orange"/>
-		</visual>
-	</link>
-	<link name="end_effector_link">
-		<visual>
-			<origin xyz="0.0 0.0 ${end_effector_length * 0.5}" rpy="0 0 0"/>
-			<geometry>
-				<box size="${end_effector_diameter} ${end_effector_diameter} ${end_effector_length}"/>
-			</geometry>
-			<material name="light_blue"/>
 		</visual>
 	</link>
@@ -71,13 +56,3 @@
 		<child link="base_link"/>
 	</joint>
-	<joint name="tool_to_end_effector" type="fixed">
-		<origin xyz="0 0 0" rpy="0 1.5708 0"/>
-		<parent link="tool0"/>
-		<child link="end_effector_link"/>
-	</joint>
-	<joint name="tool_to_tcp" type="fixed">
-		<origin xyz="${end_effector_length} 0 0" rpy="0 0 0"/>
-		<parent link="tool0"/>
-		<child link="tcp_frame"/>
-	</joint>
 </robot>

File: mtconnect_example/mtconnect_example_launch/urdf/mtconnect_m16ib20_demo_tool.urdf (robot description, URDF)
Before this commit: robot NIST_Robot, 7 links, 5 joints
Links:
- removed link base_link
- removed link cnc_link
- removed link robot_platform_link
- removed link world_frame
- link end_effector_link: geometry visual cylinder length=0.35 radius=0.05
Joints:
- removed joint platform_to_base_joint
- removed joint world_to_cnc_joint
- removed joint world_to_platform_joint

File: mtconnect_example/mtconnect_example_launch/urdf/mtconnect_m16ib20_demo_tool.xacro (robot description, xacro)
@@ -1,7 +1,5 @@
 <?xml version="1.0" ?>
 <robot name="NIST_Robot" xmlns:xacro="http://ros.org/wiki/xacro">
-	<include filename="$(find fanuc_config)/urdf/M16iB20_macro.xacro"/>
 	<!-- parameters -->
-	<xacro:property name="platform_thickness" value="0.1"/>
 	<xacro:property name="end_effector_length" value="0.35"/>
 	<xacro:property name="end_effector_diameter" value="0.1"/>
@@ -23,52 +21,18 @@
   </material>
   <!-- robot definitions, also defined in robot urdf -->
-	<link name="base_link"/>
 	<link name="tool0"/>
 	<!-- link definitions -->
-	<link name="world_frame"/>
 	<!--link name="palm"/-->
 	<link name="tcp_frame"/>
-	<link name="robot_platform_link">
-		<visual>
-			<origin xyz="0.0 0.0 -${platform_thickness * 0.5}" rpy="0 0 0"/>
-			<geometry>
-				<box size="0.5 0.5 ${platform_thickness}"/>
-			</geometry>
-			<material name="orange"/>
-		</visual>
-	</link>
 	<link name="end_effector_link">
 		<visual>
 			<origin xyz="0.0 0.0 ${end_effector_length * 0.5}" rpy="0 0 0"/>
 			<geometry>
-				<box size="${end_effector_diameter} ${end_effector_diameter} ${end_effector_length}"/>
+				<cylinder radius="${end_effector_diameter * 0.5}" length="${end_effector_length}"/>
 			</geometry>
 			<material name="light_blue"/>
 		</visual>
 	</link>
-	<link name="cnc_link">
-		<visual>
-			<geometry>
-        <mesh filename="package://mtconnect_example_launch/meshes/cnc_lathe.STL"/>
-			</geometry>
-			<material name="red"/>
-		</visual>
-	</link>
 	<!-- joint definitions -->
-	<joint name="world_to_platform_joint" type ="fixed">
-		<origin xyz="0.2 0 2" rpy="3.1417 0 0"/>
-		<parent link="world_frame"/>
-		<child link="robot_platform_link"/>
-	</joint>
-	<joint name="world_to_cnc_joint" type ="fixed">
-		<origin xyz="2.6 1.325 -0.45" rpy="1.5708 0 -1.5708"/>
-		<parent link="world_frame"/>
-		<child link="cnc_link"/>
-	</joint>
-	<joint name="platform_to_base_joint" type ="fixed">
-		<origin xyz="0 0 0" rpy="0 0 0"/>
-		<parent link="robot_platform_link"/>
-		<child link="base_link"/>
-	</joint>
 	<joint name="tool_to_end_effector" type="fixed">
 		<origin xyz="0 0 0" rpy="0 1.5708 0"/>

Commit message: Adjusted CNC offset from world frame (and base_link) to match real life.  Corrected task description with newly taught points and reordered some motions.  Updated state machine to do correct state transitions

File: mtconnect_example/mtconnect_example_launch/urdf/mtconnect_m16ib20_demo_env.urdf (robot description, URDF)
Before this commit: robot NIST_Robot, 4 links, 3 joints
Joints:
- joint world_to_cnc_joint: origin xyz=2.6 1.325 -0.45 rpy=1.5708 0 -1.5708 -> xyz=3.0 1.325 -0.45 rpy=1.5708 0 -1.5708

File: mtconnect_example/mtconnect_example_launch/urdf/mtconnect_m16ib20_demo_env.xacro (robot description, xacro)
@@ -47,5 +47,5 @@
 	</joint>
 	<joint name="world_to_cnc_joint" type ="fixed">
-		<origin xyz="2.6 1.325 -0.45" rpy="1.5708 0 -1.5708"/>
+		<origin xyz="3.0 1.325 -0.45" rpy="1.5708 0 -1.5708"/>
 		<parent link="world_frame"/>
 		<child link="cnc_link"/>

Commit message: Fixed cnc location to approximate position relative to the robot (in visualizer).  Removed unused urdf/xacro.

File: mtconnect_example/mtconnect_example_launch/urdf/mtconnect_m16ib20_demo_env.urdf (robot description, URDF)
Before this commit: robot NIST_Robot, 4 links, 3 joints
Joints:
- joint world_to_cnc_joint: origin xyz=3.0 1.325 -0.45 rpy=1.5708 0 -1.5708 -> xyz=-0.75 2.0 0 rpy=1.5708 0 0
- joint world_to_platform_joint: origin xyz=0.2 0 2 rpy=3.1417 0 0 -> xyz=0 0 3 rpy=3.1417 0 0

File: mtconnect_example/mtconnect_example_launch/urdf/mtconnect_m16ib20_demo_env.xacro (robot description, xacro)
@@ -42,10 +42,10 @@
 	<!-- joint definitions -->
 	<joint name="world_to_platform_joint" type ="fixed">
-		<origin xyz="0.2 0 2" rpy="3.1417 0 0"/>
+		<origin xyz="0 0 3" rpy="3.1417 0 0"/>
 		<parent link="world_frame"/>
 		<child link="robot_platform_link"/>
 	</joint>
 	<joint name="world_to_cnc_joint" type ="fixed">
-		<origin xyz="3.0 1.325 -0.45" rpy="1.5708 0 -1.5708"/>
+		<origin xyz="-0.75 2.0 0" rpy="1.5708 0 0"/>
 		<parent link="world_frame"/>
 		<child link="cnc_link"/>
